Commit message: Add files via upload

File: scara_description/urdf/scara copy.xacro (robot description, xacro)
@@ -13,11 +13,11 @@
     <visual>
       <geometry>
-        <box size = "0.2 0.2 0.2"/>
-      </geometry>
-      <material name = "blue"/>
-      <origin xyz = "0 0 0.1"/>
-    </visual>
-    <inertial>
-      <mass value="10" />
+        <box size = "0.12 0.12 0.05"/>
+      </geometry>
+      <material name = "blue"/>
+      <origin xyz = "0 0 0.025"/>
+    </visual>
+    <inertial>
+      <mass value="1" />
       <origin xyz="0 0 0.025" rpy="0 0 0" />
       <inertia ixx="1" ixy="0" ixz="0" iyy="1" iyz="0" izz="1" />
@@ -25,8 +25,8 @@
     <collision>
       <geometry>
-        <box size = "0.2 0.2 0.2"/>
-      </geometry>
-      <material name = "blue"/>
-      <origin xyz = "0 0 0.1"/>
+        <box size = "0.12 0.12 0.05"/>
+      </geometry>
+      <material name = "blue"/>
+      <origin xyz = "0 0 0.025"/>
     </collision>
   </link>
@@ -39,11 +39,11 @@
     <visual>
       <geometry>
-        <cylinder length = "0.160" radius = "0.09"/>
+        <cylinder length = "0.45" radius = "0.05"/>
       </geometry>
       <material name = "green"/>
-      <origin xyz = "0 0 0.08"/>
-    </visual>
-    <inertial>
-      <mass value="3.5" />
+      <origin xyz = "0 0 0.225"/>
+    </visual>
+    <inertial>
+      <mass value="0.5" />
       <origin xyz="0 0 0.05" rpy="0 0 0" />
       <inertia ixx="0.5" ixy="0" ixz="0" iyy="0.5" iyz="0" izz="0.5" />
@@ -51,15 +51,15 @@
     <collision>
       <geometry>
-        <cylinder length = "0.160" radius = "0.09"/>
+        <cylinder length = "0.45" radius = "0.05"/>
       </geometry>
       <material name = "green"/>
-      <origin xyz = "0 0 0.08"/>
-    </collision>
-  </link>
-  <joint name = "joint1" type="revolute">
+      <origin xyz = "0 0 0.225"/>
+    </collision>
+  </link>
+  <joint name = "joint1" type="continuous">
     <parent link = "base_link"/>
     <child link = "revolute1"/>
-    <origin xyz = "0 0 0.2"/>
-    <limit effort="1000.0" lower="-2.58309" upper="2.58309" velocity="7.67"/>
+    <origin xyz = "0 0 0.05"/>
+    <limit effort="1000.0" lower="-1.57" upper="1.57" velocity="0.5"/>
     <axis xyz = "0 0 1"/>
     <dynamics damping="0.2" friction="0.1" />
@@ -69,11 +69,11 @@
     <visual>
       <geometry>
-        <box size = "0.08 0.15 0.350"/>
-      </geometry>
-      <material name = "blue"/>
-      <origin rpy = "0 1.571 0" xyz = "0.175 0 0.04"/>
-    </visual>
-    <inertial>
-      <mass value="5.5" />
+        <box size = "0.1 0.1 0.425"/>
+      </geometry>
+      <material name = "blue"/>
+      <origin rpy = "0 1.571 0" xyz = "0.2125 0 0"/>
+    </visual>
+    <inertial>
+      <mass value="0.5" />
       <origin xyz="0.2125 0 0" rpy="0 0 0" />
       <inertia ixx="0.5" ixy="0" ixz="0" iyy="0.5" iyz="0" izz="0.5" />
@@ -81,8 +81,8 @@
     <collision>
       <geometry>
-        <box size = "0.08 0.15 0.350"/>
-      </geometry>
-      <material name = "blue"/>
-      <origin rpy = "0 1.571 0" xyz = "0.175 0 0.04"/>
+        <box size = "0.1 0.1 0.425"/>
+      </geometry>
+      <material name = "blue"/>
+      <origin rpy = "0 1.571 0" xyz = "0.2125 0 0"/>
     </collision>
   </link>
@@ -90,5 +90,5 @@
     <parent link = "revolute1"/>
     <child link = "link1"/>
-    <origin xyz = "0 0 0.16"/>
+    <origin xyz = "0 0 0.4"/>
   </joint>
   <!-- revolute 2 -->
@@ -96,5 +96,5 @@
     <visual>
       <geometry>
-        <cylinder length = "0.2" radius = "0.06"/>
+        <cylinder length = "0.2" radius = "0.05"/>
       </geometry>
       <material name = "green"/>
@@ -102,11 +102,11 @@
     </visual>
     <inertial>
-      <mass value="1.5" />
+      <mass value="0.5" />
       <origin xyz="0 0 0" rpy="0 0 0" />
-      <inertia ixx="0.5" ixy="0" ixz="0" iyy="0.5" iyz="0" izz="0.5" />
-    </inertial>
-    <collision>
-      <geometry>
-        <cylinder length = "0.2" radius = "0.06"/>
+      v<inertia ixx="0.5" ixy="0" ixz="0" iyy="0.5" iyz="0" izz="0.5" />
+    </inertial>
+    <collision>
+      <geometry>
+        <cylinder length = "0.2" radius = "0.05"/>
       </geometry>
       <material name = "green"/>
@@ -114,9 +114,9 @@
     </collision>
   </link>
-  <joint name = "joint2" type="revolute">
+  <joint name = "joint2" type="continuous">
     <parent link = "link1"/>
     <child link = "revolute2"/>
-    <origin xyz = "0.350 0 0.1"/>
-    <limit effort="1000.0" lower="-2.61799" upper="2.61799" velocity="12.21"/>
+    <origin xyz = "0.425 0 0.05"/>
+    <limit effort="1000.0" lower="-1.57" upper="1.57" velocity="0.5"/>
     <axis xyz = "0 0 1"/>
     <dynamics damping="0.2" friction="0.1" />
@@ -126,11 +126,11 @@
     <visual>
       <geometry>
-        <box size = "0.18 0.1 0.3"/>
-      </geometry>
-      <material name = "blue"/>
-      <origin rpy = "0 1.571 0" xyz = "0.15 0 0"/>
-    </visual>
-    <inertial>
-      <mass value="2.5" />
+        <box size = "0.1 0.1 0.345"/>
+      </geometry>
+      <material name = "blue"/>
+      <origin rpy = "0 1.571 0" xyz = "0.1725 0 0"/>
+    </visual>
+    <inertial>
+      <mass value="0.5" />
       <origin xyz="0.1725 0 0" rpy="0 0 0" />
       <inertia ixx="0.5" ixy="0" ixz="0" iyy="0.5" iyz="0" izz="0.5" />
@@ -138,8 +138,8 @@
     <collision>
       <geometry>
-        <box size = "0.18 0.1 0.3"/>
-      </geometry>
-      <material name = "blue"/>
-      <origin rpy = "0 1.571 0" xyz = "0.15 0 0"/>
+        <box size = "0.1 0.1 0.345"/>
+      </geometry>
+      <material name = "blue"/>
+      <origin rpy = "0 1.571 0" xyz = "0.1725 0 0"/>
     </collision>
   </link>
@@ -174,5 +174,5 @@
     <parent link = "link2"/>
     <child link = "prismatic3"/>
-    <origin rpy = "3.14 0 0" xyz = "0.3 0 0"/>
+    <origin rpy = "3.14 0 0" xyz = "0.345 0 0"/>
   </joint>
   <!-- link 3 -->
@@ -180,8 +180,8 @@
     <visual>
       <geometry>
-        <cylinder length = "0.425" radius = "0.02"/>
-      </geometry>
-      <material name = "blue"/>
-      <origin xyz = "0 0 -0.18"/>
+        <cylinder length = "0.5" radius = "0.03"/>
+      </geometry>
+      <material name = "blue"/>
+      <origin xyz = "0 0 -0.25"/>
     </visual>
     <inertial>
@@ -192,8 +192,8 @@
     <collision>
       <geometry>
-        <cylinder length = "0.425" radius = "0.02"/>
-      </geometry>
-      <material name = "blue"/>
-      <origin xyz = "0 0 -0.18"/>
+        <cylinder length = "0.5" radius = "0.03"/>
+      </geometry>
+      <material name = "blue"/>
+      <origin xyz = "0 0 -0.25"/>
     </collision>
   </link>
@@ -202,5 +202,5 @@
     <child link = "link3"/>
     <origin xyz = "0 0 0.11"/>
-    <limit effort="1000" lower="-0.00001" upper="0.21" velocity="2.0"/>
+    <limit effort="1000" lower="-0.00001" upper="0.3" velocity="0.1"/>
     <axis xyz = "0 0 1"/>
     <dynamics damping="0.4" friction="5" />
@@ -237,9 +237,9 @@
     </actuator>
   </transmission>
-  <!-- teble_link 1 -->
+    <!-- teble_link 1 -->
   <link name = "tlink1">
     <visual>
       <geometry>
-        <box size = "0.2 0.2 0.2"/>
+        <box size = "0.3 0.3 0.2"/>
       </geometry>
       <material name = "grey"/>
@@ -253,5 +253,5 @@
     <collision>
       <geometry>
-        <box size = "0.2 0.2 0.2"/>
+        <box size = "0.3 0.3 0.2"/>
       </geometry>
       <material name = "grey"/>
@@ -264,5 +264,5 @@
     <origin xyz = "0.5 0 0"/>
   </joint>
-  <!-- teble_link 2 -->
+    <!-- teble_link 2 -->
   <link name = "tlink2">
     <visual>
@@ -434,5 +434,5 @@
     <origin xyz = "0 0.0 0.02"/>
   </joint>
-  <link name = "object_pad4">
+    <link name = "object_pad4">
     <visual>
       <geometry>
@@ -459,9 +459,9 @@
     <child link="object_pad4"/>
     <origin xyz = "0 0.0 0.02"/>
-  </joint>
+  </joint> -->
   <!-- camera link -->
-  <xacro:property name="cameraHeight" value="0.035"/>
-  <xacro:property name="cameraLength" value="0.035"/>
-  <xacro:property name="cameraWidth" value="0.12"/>
+  <xacro:property name="cameraHeight" value="0.025"/>
+  <xacro:property name="cameraLength" value="0.025"/>
+  <xacro:property name="cameraWidth" value="0.09"/>
   <xacro:property name="cameraMass" value="0.1"/>
   <link name="camera">
